File: RAMBoard/RAMBoard.kicad_pcb (KiCad board)
At the start: 2 copper layers, 104.1 x 96.5 mm, 30 parts, among them J1 Bus_ISA_8bit, SW1 SW_DIP_x08, SW2 SW_DIP_x08, U1 AS6C4008-55PCN, U2 AS6C4008-55PCN, U3 SN74HCT138N, U4 SN74HCT138N, U5 CD74HCT30E, U6 CD74HCT30E, U7 SN74ACT245N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

Commit message: PCB texts
Parts:
- RN1, RN2: value R_Network08 -> 10K x 8
Routing:
- net A5: track 230.3 -> 82.3 mm
- net A7: track 80.9 -> 91.7 mm
- net A18: track 182.7 -> 192.9 mm
- net A8: track 66.1 -> 75.3 mm
- net A3: track 65.0 -> 73.8 mm
- net A2: track 81.1 -> 89.4 mm
- net A9: track 82.6 -> 90.2 mm
- net A13: track 85.3 -> 92.7 mm
- net A14: track 136.2 -> 143.6 mm
- net A15: track 127.1 -> 133.4 mm
- net /D6: track 99.8 -> 105.8 mm
- net /D3: track 90.2 -> 96.1 mm
- net A17: track 160.7 -> 166.4 mm
- net A16: track 172.3 -> 177.6 mm
- net A6: track 64.4 -> 69.3 mm
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Other:
- board text added: "(For use in systems with 16kB RAM on system board)"
- board text added: "1.1: 0x0000 (0-64kB) - see note"
- board text added: "1.2: 0x1000 (64-128kB)"
- board text added: "1.3: 0x2000 (128-192kB)"
- board text added: "1.4: 0x3000 (192-256kB)"
- board text added: "1.5: 0x4000 (256-320kB)"
- board text added: "1.6: 0x5000 (320-384kB)"
- board text added: "1.7: 0x6000 (384-448kB)"
- board text added: "1.8: 0x7000 (448-512kB)"
- board text added: "1MB RAM Board"
- board text added: "2.1: 0x8000 (512-576kB)"
- board text added: "2.2: 0x9000 (576-640kB)"
- board text added: "2.3: 0xA000 (640-704kB)"
- board text added: "2.4: 0xB000 (704-768kB)"
- board text added: "2.5: 0xC000 (768-832kB)"
- board text added: "2.6: 0xD000 (832-896kB)"
- board text added: "2.7: 0xE000 (896-960kB)"
- board text added: "2.8: Disables 0-16kB - see note"
- board text added: "JLCJLCJLCJLC"
- board text added: "Note: SW2.8 ON disables 0-16kB (if SW1.1 = ON)"
- board text added: "Set switches ON to enable RAM at"
- board text added: "The original design was made by Lo-tech. This is a redesign by Christian Lehner (2021) with THT parts only."
- board text added: "corresponding physical pages:"
